Commit message: urdf map fixed (root to map)

File: baby_jerry/urdf/baby_jerry.urdf (robot description, URDF)
Before this commit: robot babyjerry, 44 links, 43 joints
Links:
- added link base_link
Joints:
- added joint base_link_to_cad_root: type fixed, parent base_link, child root, origin xyz=0 0 0 rpy=0 0 0

Commit message: foxglove changes

File: baby_jerry/urdf/baby_jerry.urdf (robot description, URDF)
Before this commit: robot babyjerry, 45 links, 44 joints
Joints:
- joint base_link_to_cad_root: origin xyz=0 0 0 rpy=0 0 0 -> xyz=0 0 0 rpy=0 0 -1.570796

File: field_assembly/urdf/field_assembly.urdf (robot description, URDF)
Before this commit: robot field_assembly, 15 links, 14 joints
Links:
- added link field_origin, mass 0.000819162; visual mesh filename=file:///home/giovonnie/ghost_visualization_assets/field_ass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 scale=1 1 1; visual mesh filename=file:///home/giovonnie/ghost_visualization_assets/field_ass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 scale=1 1 1
- link map: mass 0.000819162 -> None; geometry 
Joints:
- added joint map_to_field_origin: type fixed, parent map, child field_origin, origin xyz=1.828 1.828 0 rpy=0 0 0
- joint fixed_node_to_root_joint: parent map -> field_origin
